File: HARDWARE/breakoutboard/breakoutboard.kicad_pcb (KiCad board)
At the start: 2 copper layers, 32.9 x 24.6 mm, 20 parts, among them IC1 TC1240AECHTR, IC2 LP2981-50DBVR, IC3 MIC803-30D2VM3-TR, J1 WP7B-P040VA1-R8000, J2 Conn_01x08_Pin

Commit message: dd
Parts:
- added ?: , , F.Cu at (161.4, 98.2)
- added ?: , , F.Cu at (143.9, 101.6)
- added ?: , , F.Cu at (161.4, 96.8)
- added ?: , , F.Cu at (157.3, 102.0)
- added D1: PESD2USB5UVT-QR, diode esd:SOT95P230X110-3N, F.Cu at (158.4, 105.1)
- added G***: LOGO, ensea2:logo ensea, F.Cu at (137.1, 89.0)
- added REF**: R_0402_1005Metric, Resistor_SMD:R_0402_1005Metric, F.Cu at (159.5, 96.8)
- added REF**: R_0402_1005Metric, Resistor_SMD:R_0402_1005Metric, F.Cu at (159.5, 97.9)
Routing:
- net GND: track 18.4 -> 36.6 mm, vias 67 -> 82
- net RX0: track 0.00 -> 15.5 mm, vias 0 -> 2
- net TXO: track 0.00 -> 13.3 mm, vias 0 -> 2
- net +3.3V: track 31.1 -> 27.1 mm
- net txout: track 0.00 -> 1.51 mm
- net rxout: track 0.00 -> 1.39 mm
- net +5V: track 17.3 -> 18.0 mm
- net SPI_MISO/DAT12: track 4.86 -> 5.51 mm
- net GPIO1: track 9.14 -> 9.78 mm
- net GPIO2: track 8.08 -> 8.60 mm
- net GPIO3: track 9.40 -> 9.93 mm
Other:
- board text added: "5v"
- board text added: "IO1"
- board text added: "IO2"
- board text added: "IO3"
- board text added: "rx0"
- board text added: "tx0"
