File: HARDWARE/breakoutboard/breakoutboard.kicad_sch (KiCad schematic)
At the start: 13 parts, among them IC1 TC1240AECHTR, IC2 LP2981-50DBVR, IC3 MIC803-30D2VM3-TR, J1 WP7B-P040VA1-R8000, J2 Conn_01x08_Pin

Commit message: dd
Parts:
- added D1: PESD2USB5UVT-QR, diode esd:SOT95P230X110-3N, symbol diode tvs esd:PESD2USB5UVT-QR
Connections:
- net +3.3V: now also D1.1 (K1)
- net GND: now also D1.2 (K2)
- no-connect marks 7 -> 8
