File: HARDWARE BALISE/hardware/camera_thermique_v1/camera.kicad_sch (KiCad schematic)
At the start: 12 parts, among them J1 687108183722, Q1 2N7002KQBZ

Commit message: g
Parts:
- removed R12: 100R, Resistor_SMD:R_0201_0603Metric_Pad0.64x0.40mm_HandSolder, symbol Device:R_Small
- removed R17: 1k, Resistor_SMD:R_0201_0603Metric_Pad0.64x0.40mm_HandSolder, symbol Device:R_Small
- removed R2, R6: 33R, Resistor_SMD:R_0201_0603Metric_Pad0.64x0.40mm_HandSolder, symbol Device:R_Small
- added C28: 10u, Capacitor_SMD:C_0402_1005Metric_Pad0.74x0.62mm_HandSolder, symbol Device:C_Small
- added R18: 100R, Resistor_SMD:R_0201_0603Metric_Pad0.64x0.40mm_HandSolder, symbol Device:R_Small
- Q1: value 2N7002KQBZ -> BSS84AKQBZ
Connections:
- net +3.3V: now also Q1.2 (S); no longer J1.1
- net +5V: now also C28.1
- net DATA7/SPI_CLK: now also U1.36 (DATA15/SPI_CLK)
- net GND: now also J1.2, C28.2; no longer Q1.2 (S)
- net LCD_PWM_LED: now also Q1.1 (G), R16.2
- net PIX_CLK: now also U1.33 (PIXCLK)
- net at Q1.3 (D_1), Q1.4 (D_2): now also R18.2
- new net: J1.1, R18.1
Other:
- moved on the sheet: Q1, R16
