File: HARDWARE BALISE/hardware/camera_thermique_v1/camera_thermique_v1.kicad_pcb (KiCad board)
At the start: 2 copper layers, 21.4 x 30 mm, 65 parts, among them IC1 W25Q16JWXHIQ_TR, IC2 LDO40LPU33RY, IC3 LM2775DSGT, J1 687108183722, J4 USB_C_Receptacle_USB2.0_14P, Q1 2N7002KQBZ, SW1 BOOTMODE, SW2 RESET, U2 ESP32-S3, U3 LTC4065AEDC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

Commit message: g
Parts:
- removed R12: 100R, Resistor_SMD:R_0201_0603Metric_Pad0.64x0.40mm_HandSolder
- removed R17: 1k, Resistor_SMD:R_0201_0603Metric_Pad0.64x0.40mm_HandSolder
- removed R2, R6: 33R, Resistor_SMD:R_0201_0603Metric_Pad0.64x0.40mm_HandSolder
- removed U4: USBLC6-2SC6, Package_TO_SOT_SMD:SOT-23-6
- added C28: 10u, Capacitor_SMD:C_0402_1005Metric_Pad0.74x0.62mm_HandSolder, F.Cu at (114.3, 95.7)
- added D3: 82400274, samacsys:SOT65P210X110-6N, B.Cu at (127.9, 108.6)
- added J2: 636101111001, samacsys:636101111001, B.Cu at (113.6, 108.4)
- added R18: 100R, Resistor_SMD:R_0201_0603Metric_Pad0.64x0.40mm_HandSolder, F.Cu at (115.2, 100.7)
- C1, C11, C12, C14, C15, C16, C19, C2, C20, C21, C22, C23, C24, IC1, L2, R13, R3, R8, R9, U2: moved to B.Cu
- C10, C9: value 10u -> 100n
- C17, C18: value 10u -> 1.56n; moved to B.Cu
- J1, S1, U3: moved to F.Cu
- L3: value 2.2n -> 2.7n; moved to B.Cu
- Q1: value 2N7002KQBZ -> BSS84AKQBZ
- R10, R11: value 0R -> 22R; moved to B.Cu
- Y1: value Crystal_GND24 -> 40Mhz; moved to B.Cu
- moved C26 55.4 mm to (127.2, 98.7), turned to -90 degrees
- moved R3 47.7 mm to (127.0, 112.1), turned to 180 degrees
- moved C4 46.6 mm to (126.3, 108.5)
- moved C3 45.3 mm to (120.3, 110.5), turned to 90 degrees
- moved C27 43.5 mm to (115.0, 98.2), turned to 180 degrees
- moved C25 43.3 mm to (115.0, 99.2), turned to 180 degrees
- moved R5 43.2 mm to (124.9, 111.5), turned to -90 degrees
- moved R4 42.8 mm to (126.2, 107.7), turned to 180 degrees
- moved C5 41.7 mm to (123.1, 106.7)
- moved R1 41.7 mm to (115.3, 111.5)
- moved TP1 41.5 mm to (130.7, 109.5)
- moved C13 39.3 mm to (130.2, 92.2)
- moved R14 39.1 mm to (125.4, 106.5)
- moved D2 38.5 mm to (130.6, 111.6), turned to 180 degrees
- moved Q1 38.5 mm to (113.9, 100.8), turned to -90 degrees
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Connections:
- J1 pad 1: +3.3V -> Net-(J1-Pad1)
- J1 pad 2: Net-(J1-Pad2) -> GND
- J4 pad A6: Net-(J4-D+-PadA6) -> D+
- J4 pad A7: Net-(J4-D--PadA7) -> D-
- J4 pad B6: Net-(J4-D+-PadA6) -> D+
- J4 pad B7: Net-(J4-D--PadA7) -> D-
- Q1 pad 1: Net-(Q1-G) -> LCD_PWM_LED
- Q1 pad 2: GND -> +3.3V
- R16 pad 2: Net-(Q1-G) -> LCD_PWM_LED
- U1 pad 33: Net-(U1-PIXCLK) -> PIX_CLK
- U1 pad 36: Net-(U1-DATA15/SPI_CLK) -> DATA7/SPI_CLK
- U2 pad 10: unconnected-(U2-GPIO5-Pad10) -> LCD_PWM_LED
- U2 pad 12: DATA1 -> DATA3
- U2 pad 14: DATA3 -> DATA1
- U2 pad 19: VSYNC -> PIX_CLK
- U2 pad 23: HSYNC -> VSYNC
- U2 pad 24: PIX_CLK -> HSYNC
- U2 pad 27: LCD_PWM_LED -> unconnected-(U2-GPIO21-Pad27)
- U2 pad 38: LCD_RES -> LCD_CS
- U2 pad 39: LCD_DC -> LCD_CLK
- U2 pad 41: LCD_CLK -> LCD_MOSI
- U2 pad 42: LCD_CS -> LCD_DC
- U2 pad 43: LCD_MOSI -> LCD_RES
- U2 pad 57: unconnected-(U2-GND-Pad57) -> GND
Routing:
- net Net-(D1-A): track 0.00 -> 39.0 mm, vias 0 -> 6
- net +3.3V: track 0.00 -> 25.3 mm, vias 0 -> 13
- net vusb: track 0.00 -> 20.4 mm, vias 0 -> 5
- net BOOT0: track 0.00 -> 19.6 mm, vias 0 -> 2
- net Net-(U2-GPIO19/USB_D-): track 0.00 -> 16.0 mm, vias 0 -> 2
- net GND: track 0.00 -> 15.8 mm, vias 0 -> 61
- net Net-(U2-GPIO20/USB_D+): track 0.00 -> 14.4 mm, vias 0 -> 2
- net VBAT+: track 0.00 -> 13.6 mm, vias 0 -> 1
- net BAT+: track 0.00 -> 10.4 mm
- net CAM_SCL: track 0.00 -> 10.3 mm, vias 0 -> 2
- net SPICS0: track 0.00 -> 9.65 mm, vias 0 -> 2
- net SPIQ: track 0.00 -> 9.01 mm, vias 0 -> 2
- net Net-(U2-LNA_IN): track 0.00 -> 8.30 mm
- net SPIWP: track 0.00 -> 7.80 mm, vias 0 -> 2
- net LCD_PWM_LED: track 0.00 -> 7.44 mm, vias 0 -> 2
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- added copper zone on B.Cu, net +3.3V
- added copper zone on F.Cu, net +3.3V
- added copper zone on F.Cu, net +5V
- added copper zone on F.Cu, net BAT+
- added copper zone on F.Cu, net BOOT0
- added copper zone on B.Cu, net GND
- added copper zone on F.Cu, net GND
- added copper zone on In3.Cu, net GND
- added copper zone on F.Cu, net Net-(D1-A)
- added copper zone on F.Cu, net VBAT+
- added copper zone on F.Cu, net vusb
Other:
- board size 21.4 x 30 mm -> 21.4 x 33.5 mm
- copper layers 2 -> 6
