File: HARDWARE BALISE/hardware/camera_thermique_v1/camera_thermique_v1.kicad_sch (KiCad schematic)
At the start: 28 parts, among them IC1 W25Q16JWXHIQ_TR, SW1 BOOTMODE, SW2 RESET, U2 ESP32-S3, Y1 Crystal_GND24

Commit message: g
Parts:
- added J2: 636101111001, 636101111001, symbol samacsys:636101111001
- C17, C18: value 10u -> 1.56n
- L3: value 2.2n -> 2.7n
- R10, R11: value 0R -> 22R
- Y1: value Crystal_GND24 -> 40Mhz
Connections:
- net ANT: now also J2.3
- net DATA1: now also U2.14 (GPIO9); no longer U2.12 (GPIO7)
- net DATA3: now also U2.12 (GPIO7); no longer U2.14 (GPIO9)
- net GND: now also U2.57 (GND), J2.1, J2.2
- net HSYNC: now also U2.24 (GPIO18); no longer U2.23 (GPIO17)
- net LCD_CLK: now also U2.39 (GPIO34); no longer U2.41 (GPIO36)
- net LCD_CS: now also U2.38 (GPIO33); no longer U2.42 (GPIO37)
- net LCD_DC: now also U2.42 (GPIO37); no longer U2.39 (GPIO34)
- net LCD_MOSI: now also U2.41 (GPIO36); no longer U2.43 (GPIO38)
- net LCD_PWM_LED: now also U2.10 (GPIO5); no longer U2.27 (GPIO21)
- net LCD_RES: now also U2.43 (GPIO38); no longer U2.38 (GPIO33)
- net PIX_CLK: now also U2.19 (GPIO14); no longer U2.24 (GPIO18)
- net VSYNC: now also U2.23 (GPIO17); no longer U2.19 (GPIO14)
