File: HARDWARE BALISE/hardware/camera_thermique_v1/power.kicad_sch (KiCad schematic)
At the start: 25 parts, among them IC2 LDO40LPU33RY, IC3 LM2775DSGT, J4 USB_C_Receptacle_USB2.0_14P, U3 LTC4065AEDC, U4 USBLC6-2SC6

Commit message: g
Parts:
- removed U4: USBLC6-2SC6, Package_TO_SOT_SMD:SOT-23-6, symbol Power_Protection:USBLC6-2SC6
- added D3: 82400274, SOT65P210X110-6N, symbol samacsys:82400274
- C10, C9: value 10u -> 100n
Connections:
- net D+: now also J4.A6 (D+), J4.B6 (D+), D3.4 (I/O_3)
- net D-: now also J4.A7 (D-), J4.B7 (D-), D3.6 (I/O_4)
- net GND: now also D3.2 (GND)
- net vusb: now also D3.5 (VDD)
Changed lines of the file:
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@@
 	(rectangle
 		(start 294.64 113.03)
-		(end 396.24 189.23)
+		(end 406.4 200.66)
 		(stroke
 			(width 0)
@@
 	)
 	(no_connect
-		(at 355.6 163.83)
+		(at 363.22 185.42)
 	)
 	(no_connect
-		(at 355.6 160.02)
+		(at 363.22 190.5)
 	)
 	(no_connect
@@
 	(wire
 		(pts
-			(xy 374.65 157.48) (xy 374.65 156.21)
-		)
-		(stroke
-			(width 0)
-			(type default)
-		)
-	)
-	(wire
-		(pts
 			(xy 50.8 186.69) (xy 62.23 186.69)
 		)
@@
 	(global_label "D-"
 		(shape input)
-		(at 379.73 162.56 0)
+		(at 369.57 162.56 0)
+		(fields_autoplaced yes)
+		(effects
+			(font
+				(size 1.27 1.27)
+			)
+			(justify left)
+		)
+		(property "Intersheetrefs" "${INTERSHEET_REFS}"
+			(at 375.3976 162.56 0)
+			(effects
+				(font
+					(size 1.27 1.27)
+				)
+				(justify left)
+				(hide yes)
+			)
+		)
+	)
+	(global_label "D-"
+		(shape input)
+		(at 393.7 185.42 0)
 		(fields_autoplaced yes)
 		(effects
@@
 		)
 		(property "Intersheetrefs" "${INTERSHEET_REFS}"
-			(at 385.5576 162.56 0)
+			(at 399.5276 185.42 0)
+			(effects
+				(font
+					(size 1.27 1.27)
+				)
+				(justify left)
+				(hide yes)
+			)
+		)
+	)
+	(global_label "D+"
+		(shape input)
+		(at 393.7 190.5 0)
+		(fields_autoplaced yes)
+		(effects
+			(font
+				(size 1.27 1.27)
+			)
+			(justify left)
+		)
+		(property "Intersheetrefs" "${INTERSHEET_REFS}"
+			(at 399.5276 190.5 0)
 			(effects
 				(font
@@
 	(global_label "vusb"
 		(shape input)
-		(at 374.65 156.21 90)
+		(at 393.7 187.96 0)
 		(fields_autoplaced yes)
 		(effects
@@
 		)
 		(property "Intersheetrefs" "${INTERSHEET_REFS}"
-			(at 374.65 148.9311 90)
+			(at 400.9789 187.96 0)
 			(effects
 				(font
@@
 	(global_label "D+"
 		(shape input)
-		(at 379.73 165.1 0)
+		(at 369.57 165.1 0)
 		(fields_autoplaced yes)
 		(effects
@@
 		)
 		(property "Intersheetrefs" "${INTERSHEET_REFS}"
-			(at 385.5576 165.1 0)
+			(at 375.3976 165.1 0)
 			(effects
 				(font
@@
 			)
 		)
-		(property "Value" "10u"
+		(property "Value" "100n"
 			(at 358.14 72.3962 0)
 			(effects
@@
 	)
 	(symbol
-		(lib_id "Power_Protection:USBLC6-2SC6")
-		(at 374.65 162.56 0)
-		(unit 1)
-		(exclude_from_sim no)
-		(in_bom yes)
-		(on_board yes)
-		(dnp no)
-		(fields_autoplaced yes)
-		(property "Reference" "U4"
-			(at 376.3011 154.94 0)
-			(effects
-				(font
-					(size 1.27 1.27)
-				)
-				(justify left)
-			)
-		)
-		(property "Value" "USBLC6-2SC6"
-			(at 376.3011 157.48 0)
-			(effects
-				(font
-					(size 1.27 1.27)
-				)
-				(justify left)
-			)
-		)
-		(property "Footprint" "Package_TO_SOT_SMD:SOT-23-6"
-			(at 375.92 168.91 0)
-			(effects
-				(font
-					(size 1.27 1.27)
-					(italic yes)
-				)
-				(justify left)
-				(hide yes)
-			)
-		)
-		(property "Datasheet" "https://www.st.com/resource/en/datasheet/usblc6-2.pdf"
-			(at 375.92 170.815 0)
-			(effects
-				(font
-					(size 1.27 1.27)
-				)
-				(justify left)
-				(hide yes)
-			)
-		)
-		(property "Description" "Very low capacitance ESD protection diode, 2 data-line, SOT-23-6"
-			(at 374.65 162.56 0)
-			(effects
-				(font
-					(size 1.27 1.27)
-				)
-				(hide yes)
-			)
-		)
-		(pin "2"
-		)
-		(pin "6"
-		)
-		(pin "5"
-		)
-		(pin "3"
-		)
-		(pin "4"
-		)
-		(pin "1"
-		)
-		(instances
-			(project "camera_thermique_v1"
-				(path "/b4bd77eb-325c-489e-9021-f102496f9919/d5d5d3c6-b6e4-40a4-9ae2-23d7b657860d"
-					(reference "U4")
-					(unit 1)
-				)
-			)
-		)
-	)
-	(symbol
 		(lib_id "power:+5V")
 		(at 379.73 68.58 0)
@@
 	)
 	(symbol
+		(lib_id "samacsys:82400274")
+		(at 363.22 185.42 0)
+		(unit 1)
+		(exclude_from_sim no)
+		(in_bom yes)
+		(on_board yes)
+		(dnp no)
+		(fields_autoplaced yes)
+		(property "Reference" "D3"
+			(at 378.46 177.8 0)
+			(effects
+				(font
+					(size 1.27 1.27)
+				)
+			)
+		)
+		(property "Value" "82400274"
+			(at 378.46 180.34 0)
+			(effects
+				(font
+					(size 1.27 1.27)
+				)
+			)
+		)
+		(property "Footprint" "SOT65P210X110-6N"
+			(at 389.89 280.34 0)
+			(effects
+				(font
+					(size 1.27 1.27)
+				)
+				(justify left top)
+				(hide yes)
+			)
+		)
+		(property "Datasheet" "https://katalog.we-online.com/pbs/datasheet/82400274.pdf"
+			(at 389.89 380.34 0)
+			(effects
+				(font
+					(size 1.27 1.27)
+				)
+				(justify left top)
+				(hide yes)
+			)
+		)
+		(property "Description" "TVS Diode Array WE-TVS 4-Ch+VDD 5V SC70 Wurth Elektronik 82400274, Quad Uni-Directional TVS Diode Array, 6-Pin SC-70"
+			(at 363.22 185.42 0)
+			(effects
+				(font
+					(size 1.27 1.27)
+				)
+				(hide yes)
+			)
+		)
+		(property "Height" "1.1"
+			(at 389.89 580.34 0)
+			(effects
+				(font
+					(size 1.27 1.27)
+				)
+				(justify left top)
+				(hide yes)
+			)
+		)
+		(property "Mouser Part Number" "710-82400274"
+			(at 389.89 680.34 0)
+			(effects
+				(font
+					(size 1.27 1.27)
+				)
+				(justify left top)
+				(hide yes)
+			)
+		)
+		(property "Mouser Price/Stock" "https://www.mouser.co.uk/ProductDetail/Wurth-Elektronik/82400274?qs=2kOmHSv6VfQD871MY%252BLLLQ%3D%3D"
+			(at 389.89 780.34 0)
+			(effects
+				(font
+					(size 1.27 1.27)
+				)
+				(justify left top)
+				(hide yes)
+			)
+		)
+		(property "Manufacturer_Name" "Wurth Elektronik"
+			(at 389.89 880.34 0)
+			(effects
+				(font
+					(size 1.27 1.27)
+				)
+				(justify left top)
+				(hide yes)
+			)
+		)
+		(property "Manufacturer_Part_Number" "82400274"
+			(at 389.89 980.34 0)
+			(effects
+				(font
+					(size 1.27 1.27)
+				)
+				(justify left top)
+				(hide yes)
+			)
+		)
+		(pin "3"
+		)
+		(pin "5"
+		)
+		(pin "2"
+		)
+		(pin "4"
+		)
+		(pin "1"
+		)
+		(pin "6"
+		)
+		(instances
+			(project ""
+				(path "/b4bd77eb-325c-489e-9021-f102496f9919/d5d5d3c6-b6e4-40a4-9ae2-23d7b657860d"
+					(reference "D3")
+					(unit 1)
+				)
+			)
+		)
+	)
+	(symbol
 		(lib_id "Device:C_Small")
 		(at 306.07 71.12 0)
@@
 			)
 		)
-		(property "Value" "10u"
+		(property "Value" "100n"
 			(at 337.82 72.3962 0)
 			(effects
@@
 	(symbol
 		(lib_id "power:GND")
-		(at 374.65 170.18 0)
+		(at 363.22 187.96 270)
 		(unit 1)
 		(exclude_from_sim no)
@@
 		(fields_autoplaced yes)
 		(property "Reference" "#PWR026"
-			(at 374.65 176.53 0)
+			(at 356.87 187.96 0)
 			(effects
 				(font
@@
 		)
 		(property "Value" "GND"
-			(at 374.65 175.26 0)
+			(at 359.41 187.9599 90)
 			(effects
 				(font
 					(size 1.27 1.27)
 				)
+				(justify right)
 			)
 		)
 		(property "Footprint" ""
-			(at 374.65 170.18 0)
+			(at 363.22 187.96 0)
 			(effects
 				(font
@@
 		)
 		(property "Datasheet" ""
-			(at 374.65 170.18 0)
+			(at 363.22 187.96 0)
 			(effects
 				(font
@@
 		)
 		(property "Description" "Power symbol creates a global label with name \"GND\" , ground"
-			(at 374.65 170.18 0)
+			(at 363.22 187.96 0)
 			(effects
 				(font
